File: sol_inv/mcu_power.kicad_sch (KiCad schematic)
At the start: 16 parts, among them SW1 SW_Push_Dual, U9 PSC3M5_E-LQFP-64

Commit message: v0.2 components change + reference to providers
Parts:
- C10: renamed from C8; footprint Capacitor_SMD:C_1206_3216Metric -> Capacitor_SMD:C_0603_1608Metric; ComponentLink2URL (none) -> https://ro.farnell.com/samsung-electro-mechanics/cl10a106kp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
- C11: renamed from C9; footprint Capacitor_SMD:C_1206_3216Metric -> Capacitor_SMD:C_0603_1608Metric; ComponentLink2URL (none) -> https://ro.farnell.com/samsung-electro-mechanics/cl10a106kp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
- C12: renamed from C10; footprint Capacitor_SMD:C_1206_3216Metric -> Capacitor_SMD:C_0603_1608Metric; ComponentLink2URL (none) -> https://ro.farnell.com/samsung-electro-mechanics/cl10a106kp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
- C13: renamed from C11; footprint Capacitor_SMD:C_1206_3216Metric -> Capacitor_SMD:C_0201_0603Metric; ComponentLink2URL (none) -> https://ro.farnell.com/wurth-elektronik/885012104002/cap-0-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
- C14: renamed from C12; footprint Capacitor_SMD:C_1206_3216Metric -> Capacitor_SMD:C_0201_0603Metric; ComponentLink2URL (none) -> https://ro.farnell.com/wurth-elektronik/885012104002/cap-0-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
- C15: renamed from C13; footprint Capacitor_SMD:C_1206_3216Metric -> Capacitor_SMD:C_0201_0603Metric; ComponentLink2URL (none) -> https://ro.farnell.com/wurth-elektronik/885012104002/cap-0-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
- C16: renamed from C14; footprint Capacitor_SMD:C_1206_3216Metric -> Capacitor_SMD:C_0201_0603Metric; ComponentLink2URL (none) -> https://ro.farnell.com/wurth-elektronik/885012104002/cap-0-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
- C17: renamed from C15; footprint Capacitor_SMD:C_1206_3216Metric -> Capacitor_SMD:C_0201_0603Metric; ComponentLink2URL (none) -> https://ro.farnell.com/wurth-elektronik/885012104002/cap-0-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
- C18: renamed from C16; footprint Capacitor_SMD:C_1206_3216Metric -> Capacitor_SMD:C_0201_0603Metric; ComponentLink2URL (none) -> https://ro.farnell.com/wurth-elektronik/885012104002/cap-0-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
- C19: renamed from C17; footprint Capacitor_SMD:C_1206_3216Metric -> Capacitor_SMD:C_0402_1005Metric; ComponentLink2URL (none) -> https://ro.farnell.com/taiyo-yuden/msase105sb7224kfnb25/cap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
- C20: renamed from C18; footprint Capacitor_SMD:C_1206_3216Metric -> Capacitor_SMD:C_0402_1005Metric; ComponentLink2URL (none) -> https://ro.farnell.com/yageo/cc0402krx5r6bb475/cap-4-7uf-10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
- C9: renamed from C7; footprint Capacitor_SMD:C_1206_3216Metric -> Capacitor_SMD:C_0603_1608Metric; ComponentLink2URL (none) -> https://ro.farnell.com/samsung-electro-mechanics/cl10a106kp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
- R16: footprint Resistor_SMD:R_1206_3216Metric -> Resistor_SMD:R_2010_5025Metric; ComponentLink2URL (none) -> https://ro.farnell.com/multicomp-pro/mpp102wj010jt2e/res-1r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
- R17: ComponentLink2URL (none) -> https://ro.farnell.com/multicomp-pro/mcmr04x4701ftl/res-4k7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
- SW1: ComponentLink2URL (none) -> https://ro.mouser.com/ProductDetail/Omron-Electronics/B3F-1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
- U9: ComponentLink2URL (none) -> https://ro.farnell.com/infineon/psc3m5fds2acq1xqla1/mcu-32b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

Commit message: initial component placement
Connections:
- net GNDD: now also SW1.3; no longer SW1.2
- net ~{XRES}: now also SW1.2; no longer SW1.3
Other:
- moved on the sheet: SW1
Changed lines of the file:
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@@
 	(title_block
 		(title "MCU Power Delivery")
-		(date "2025-04-10")
-		(rev "0.2")
+		(date "2025-04-24")
+		(rev "0.2.1")
 		(company "Cezar-Octavian Bontaș")
 	)
@@
 	)
 	(junction
+		(at 40.64 173.99)
+		(diameter 0)
+		(color 0 0 0 0)
+	)
+	(junction
 		(at 44.45 86.36)
 		(diameter 0)
@@
 	)
 	(junction
-		(at 43.18 149.86)
+		(at 45.72 149.86)
 		(diameter 0)
 		(color 0 0 0 0)
@@
 	)
 	(junction
-		(at 40.64 167.64)
-		(diameter 0)
-		(color 0 0 0 0)
-	)
-	(junction
 		(at 166.37 86.36)
 		(diameter 0)
@@
 	(wire
 		(pts
-			(xy 38.1 154.94) (xy 38.1 149.86)
-		)
-		(stroke
-			(width 0)
-			(type default)
-		)
-	)
-	(wire
-		(pts
 			(xy 166.37 93.98) (xy 166.37 96.52)
 		)
@@
 	(wire
 		(pts
+			(xy 45.72 149.86) (xy 55.88 149.86)
+		)
+		(stroke
+			(width 0)
+			(type default)
+		)
+	)
+	(wire
+		(pts
 			(xy 30.48 67.31) (xy 30.48 60.96)
 		)
@@
 	(wire
 		(pts
-			(xy 40.64 167.64) (xy 40.64 176.53)
+			(xy 40.64 173.99) (xy 40.64 182.88)
 		)
 		(stroke
@@
 	(wire
 		(pts
+			(xy 45.72 149.86) (xy 45.72 160.02)
+		)
+		(stroke
+			(width 0)
+			(type default)
+		)
+	)
+	(wire
+		(pts
 			(xy 30.48 96.52) (xy 30.48 95.25)
 		)
@@
 	(wire
 		(pts
+			(xy 35.56 165.1) (xy 35.56 173.99)
+		)
+		(stroke
+			(width 0)
+			(type default)
+		)
+	)
+	(wire
+		(pts
 			(xy 30.48 102.87) (xy 40.64 102.87)
 		)
@@
 	(wire
 		(pts
-			(xy 40.64 167.64) (xy 43.18 167.64)
+			(xy 40.64 173.99) (xy 45.72 173.99)
 		)
 		(stroke
@@
 	(wire
 		(pts
+			(xy 35.56 149.86) (xy 35.56 160.02)
+		)
+		(stroke
+			(width 0)
+			(type default)
+		)
+	)
+	(wire
+		(pts
 			(xy 21.59 102.87) (xy 30.48 102.87)
 		)
@@
 	(wire
 		(pts
-			(xy 38.1 167.64) (xy 40.64 167.64)
-		)
-		(stroke
-			(width 0)
-			(type default)
-		)
-	)
-	(wire
-		(pts
 			(xy 76.2 95.25) (xy 76.2 78.74)
 		)
@@
 	(wire
 		(pts
-			(xy 43.18 154.94) (xy 43.18 149.86)
-		)
-		(stroke
-			(width 0)
-			(type default)
-		)
-	)
-	(wire
-		(pts
 			(xy 21.59 54.61) (xy 30.48 54.61)
 		)
@@
 	(wire
 		(pts
-			(xy 40.64 149.86) (xy 43.18 149.86)
+			(xy 40.64 149.86) (xy 45.72 149.86)
+		)
+		(stroke
+			(width 0)
+			(type default)
+		)
+	)
+	(wire
+		(pts
+			(xy 35.56 173.99) (xy 40.64 173.99)
 		)
 		(stroke
@@
 	(wire
 		(pts
+			(xy 45.72 165.1) (xy 45.72 173.99)
+		)
+		(stroke
+			(width 0)
+			(type default)
+		)
+	)
+	(wire
+		(pts
 			(xy 21.59 91.44) (xy 21.59 102.87)
 		)
@@
 	(wire
 		(pts
-			(xy 43.18 167.64) (xy 43.18 165.1)
-		)
-		(stroke
-			(width 0)
-			(type default)
-		)
-	)
-	(wire
-		(pts
 			(xy 166.37 86.36) (xy 168.91 86.36)
 		)
@@
 	(wire
 		(pts
-			(xy 38.1 149.86) (xy 40.64 149.86)
-		)
-		(stroke
-			(width 0)
-			(type default)
-		)
-	)
-	(wire
-		(pts
-			(xy 43.18 149.86) (xy 55.88 149.86)
+			(xy 35.56 149.86) (xy 40.64 149.86)
 		)
 		(stroke
@@
 		(pts
 			(xy 36.83 73.66) (xy 36.83 86.36)
-		)
-		(stroke
-			(width 0)
-			(type default)
-		)
-	)
-	(wire
-		(pts
-			(xy 38.1 165.1) (xy 38.1 167.64)
 		)
 		(stroke
@@
 	(symbol
 		(lib_id "Switch:SW_Push_Dual")
-		(at 40.64 160.02 270)
+		(at 40.64 162.56 0)
 		(unit 1)
 		(exclude_from_sim no)
@@
 		(dnp no)
 		(property "Reference" "SW1"
-			(at 35.56 158.7499 90)
+			(at 39.3699 167.64 90)
 			(effects
 				(font
@@
 		)
 		(property "Value" "SW_Push_Dual"
-			(at 35.56 161.2899 90)
+			(at 41.9099 167.64 90)
 			(effects
 				(font
@@
 		)
 		(property "Footprint" "B3F-1000:SW_B3F-1000_OMR"
-			(at 48.26 160.02 0)
+			(at 40.64 154.94 0)
 			(effects
 				(font
@@
 		)
 		(property "Datasheet" "https://ro.mouser.com/datasheet/2/307/en_b3f-1664344.pdf"
-			(at 40.64 160.02 0)
+			(at 40.64 162.56 0)
 			(effects
 				(font
@@
 		)
 		(property "Description" "Push button switch, generic, symbol, four pins"
-			(at 40.64 160.02 0)
+			(at 40.64 162.56 0)
 			(effects
 				(font
@@
 		)
 		(property "ComponentLink1URL" ""
-			(at 40.64 160.02 0)
+			(at 40.64 162.56 0)
 			(effects
 				(font
@@
 		)
 		(property "ComponentLink2URL" "https://ro.mouser.com/ProductDetail/Omron-Electronics/B3F-1000?qs=lK7M36XCk6JQHckSc1xIsg%3D%3D"
-			(at 40.64 160.02 0)
+			(at 40.64 162.56 0)
 			(effects
 				(font
@@
 	(symbol
 		(lib_id "power:GNDD")
-		(at 40.64 176.53 0)
+		(at 40.64 182.88 0)
 		(unit 1)
 		(exclude_from_sim no)
@@
 		(fields_autoplaced yes)
 		(property "Reference" "#PWR030"
+			(at 40.64 189.23 0)
+			(effects
+				(font
+					(size 1.27 1.27)
+				)
+				(hide yes)
+			)
+		)
+		(property "Value" "GNDD"
+			(at 40.64 186.69 0)
+			(effects
+				(font
+					(size 1.27 1.27)
+				)
+			)
+		)
+		(property "Footprint" ""
 			(at 40.64 182.88 0)
 			(effects
@@
 			)
 		)
-		(property "Value" "GNDD"
-			(at 40.64 180.34 0)
-			(effects
-				(font
-					(size 1.27 1.27)
-				)
-			)
-		)
-		(property "Footprint" ""
-			(at 40.64 176.53 0)
-			(effects
-				(font
-					(size 1.27 1.27)
-				)
-				(hide yes)
-			)
-		)
 		(property "Datasheet" ""
-			(at 40.64 176.53 0)
+			(at 40.64 182.88 0)
 			(effects
 				(font
@@
 		)
 		(property "Description" "Power symbol creates a global label with name \"GNDD\" , digital ground"
-			(at 40.64 176.53 0)
-			(effects
-				(font
+			(at 40.64 182.88 0)
+			(effects
+				(font

Commit message: v0.3 pcb layout pre-drc fixes
Parts:
- C13, C14, C15, C16, C17, C18: footprint Capacitor_SMD:C_0201_0603Metric -> Capacitor_SMD:C_0402_1005Metric; ComponentLink2URL https://ro.farnell.com/wurth-elektronik/885012104002/cap-0-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 -> https://ro.farnell.com/kemet/c0402c104k4ractu/cap-0-1-f-16v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
- R16: footprint Resistor_SMD:R_2010_5025Metric -> Resistor_SMD:R_0603_1608Metric; ComponentLink2URL https://ro.farnell.com/multicomp-pro/mpp102wj010jt2e/res-1r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 -> https://ro.farnell.com/panasonic/erjup3j1r0v/res-1r-5-0-25w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
Changed lines of the file:
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@@
 	(title_block
 		(title "MCU Power Delivery")
-		(date "2025-04-24")
-		(rev "0.2.1")
+		(date "2025-05-01")
+		(rev "0.3")
 		(company "Cezar-Octavian Bontaș")
 	)
@@
 			)
 		)
-		(property "Footprint" "Capacitor_SMD:C_0201_0603Metric"
+		(property "Footprint" "Capacitor_SMD:C_0402_1005Metric"
 			(at 44.45 69.85 0)
 			(effects
@@
 			)
 		)
-		(property "Datasheet" "https://www.farnell.com/datasheets/3816100.pdf"
+		(property "Datasheet" "https://content.kemet.com/datasheets/KEM_C1002_X7R_SMD.pdf"
 			(at 44.45 69.85 0)
 			(effects
@@
 			)
 		)
-		(property "ComponentLink2URL" "https://ro.farnell.com/wurth-elektronik/885012104002/cap-0-1uf-10v-mlcc-0201/dp/4137872"
+		(property "ComponentLink2URL" "https://ro.farnell.com/kemet/c0402c104k4ractu/cap-0-1-f-16v-10-x7r-0402/dp/1288252"
 			(at 44.45 69.85 0)
 			(effects
@@
 			)
 		)
-		(property "Footprint" "Capacitor_SMD:C_0201_0603Metric"
+		(property "Footprint" "Capacitor_SMD:C_0402_1005Metric"
 			(at 55.88 158.75 0)
 			(effects
@@
 			)
 		)
-		(property "Datasheet" "https://www.farnell.com/datasheets/3816100.pdf"
+		(property "Datasheet" "https://content.kemet.com/datasheets/KEM_C1002_X7R_SMD.pdf"
 			(at 55.88 158.75 0)
 			(effects
@@
 			)
 		)
-		(property "ComponentLink2URL" "https://ro.farnell.com/wurth-elektronik/885012104002/cap-0-1uf-10v-mlcc-0201/dp/4137872"
+		(property "ComponentLink2URL" "https://ro.farnell.com/kemet/c0402c104k4ractu/cap-0-1-f-16v-10-x7r-0402/dp/1288252"
 			(at 55.88 158.75 0)
 			(effects
@@
 			)
 		)
-		(property "Footprint" "Capacitor_SMD:C_0201_0603Metric"
+		(property "Footprint" "Capacitor_SMD:C_0402_1005Metric"
 			(at 40.64 31.75 0)
 			(effects
@@
 			)
 		)
-		(property "Datasheet" "https://www.farnell.com/datasheets/3816100.pdf"
+		(property "Datasheet" "https://content.kemet.com/datasheets/KEM_C1002_X7R_SMD.pdf"
 			(at 40.64 31.75 0)
 			(effects
@@
 			)
 		)
-		(property "ComponentLink2URL" "https://ro.farnell.com/wurth-elektronik/885012104002/cap-0-1uf-10v-mlcc-0201/dp/4137872"
+		(property "ComponentLink2URL" "https://ro.farnell.com/kemet/c0402c104k4ractu/cap-0-1-f-16v-10-x7r-0402/dp/1288252"
 			(at 40.64 31.75 0)
 			(effects
@@
 			)
 		)
-		(property "Footprint" "Resistor_SMD:R_2010_5025Metric"
+		(property "Footprint" "Resistor_SMD:R_0603_1608Metric"
 			(at 19.812 87.63 90)
 			(effects
@@
 			)
 		)
-		(property "Datasheet" "https://www.farnell.com/datasheets/3990272.pdf"
+		(property "Datasheet" "https://www.farnell.com/datasheets/3156916.pdf"
 			(at 21.59 87.63 0)
 			(effects
@@
 			)
 		)
-		(property "ComponentLink2URL" "https://ro.farnell.com/multicomp-pro/mpp102wj010jt2e/res-1r-5-200v-thick-film-2010/dp/4229008"
+		(property "ComponentLink2URL" "https://ro.farnell.com/panasonic/erjup3j1r0v/res-1r-5-0-25w-0603/dp/3579433"
 			(at 21.59 87.63 0)
 			(effects
@@
 			)
 		)
-		(property "Footprint" "Capacitor_SMD:C_0201_0603Metric"
+		(property "Footprint" "Capacitor_SMD:C_0402_1005Metric"
 			(at 40.64 99.06 0)
 			(effects
@@
 			)
 		)
-		(property "Datasheet" "https://www.farnell.com/datasheets/3816100.pdf"
+		(property "Datasheet" "https://content.kemet.com/datasheets/KEM_C1002_X7R_SMD.pdf"
 			(at 40.64 99.06 0)
 			(effects
@@
 			)
 		)
-		(property "ComponentLink2URL" "https://ro.farnell.com/wurth-elektronik/885012104002/cap-0-1uf-10v-mlcc-0201/dp/4137872"
+		(property "ComponentLink2URL" "https://ro.farnell.com/kemet/c0402c104k4ractu/cap-0-1-f-16v-10-x7r-0402/dp/1288252"
 			(at 40.64 99.06 0)
 			(effects
@@
 			)
 		)
-		(property "Footprint" "Capacitor_SMD:C_0201_0603Metric"
+		(property "Footprint" "Capacitor_SMD:C_0402_1005Metric"
 			(at 44.45 82.55 0)
 			(effects
@@
 			)
 		)
-		(property "Datasheet" "https://www.farnell.com/datasheets/3816100.pdf"
+		(property "Datasheet" "https://content.kemet.com/datasheets/KEM_C1002_X7R_SMD.pdf"
 			(at 44.45 82.55 0)
 			(effects
@@
 			)
 		)
-		(property "ComponentLink2URL" "https://ro.farnell.com/wurth-elektronik/885012104002/cap-0-1uf-10v-mlcc-0201/dp/4137872"
+		(property "ComponentLink2URL" "https://ro.farnell.com/kemet/c0402c104k4ractu/cap-0-1-f-16v-10-x7r-0402/dp/1288252"
 			(at 44.45 82.55 0)
 			(effects
@@
 			)
 		)
-		(property "Footprint" "Capacitor_SMD:C_0201_0603Metric"
+		(property "Footprint" "Capacitor_SMD:C_0402_1005Metric"
 			(at 40.64 50.8 0)
 			(effects
@@
 			)
 		)
-		(property "Datasheet" "https://www.farnell.com/datasheets/3816100.pdf"
+		(property "Datasheet" "https://content.kemet.com/datasheets/KEM_C1002_X7R_SMD.pdf"
 			(at 40.64 50.8 0)
 			(effects
@@
 			)
 		)
-		(property "ComponentLink2URL" "https://ro.farnell.com/wurth-elektronik/885012104002/cap-0-1uf-10v-mlcc-0201/dp/4137872"
+		(property "ComponentLink2URL" "https://ro.farnell.com/kemet/c0402c104k4ractu/cap-0-1-f-16v-10-x7r-0402/dp/1288252"
 			(at 40.64 50.8 0)
 			(effects
